Commit message: Actualizacion mundo, carro y posiciones del lidar y la camara

File: simulacion_ws/src/carro_simulacion/urdf/carro.urdf (robot description, URDF)
Before this commit: robot Carros, 10 links, 9 joints
Joints:
- joint camera_joint: origin xyz=-0.02 0 0.11 rpy=0 0 0 -> xyz=-0.02 0 0.10 rpy=0 0 0
- joint lidar_joint: origin xyz=-0.08 0 0.12 rpy=0 0 0 -> xyz=-0.15 0 0.07 rpy=0 0 0

Commit message: Actualizacion

File: simulacion_ws/src/carro_simulacion/urdf/carro.urdf (robot description, URDF)
Before this commit: robot Carros, 10 links, 9 joints
Joints:
- joint camera_joint: origin xyz=-0.02 0 0.10 rpy=0 0 0 -> xyz=-0.02 0 0.125 rpy=0 0 0

Commit message: Actualizacion

File: simulacion_ws/src/carro_simulacion/urdf/carro.urdf (robot description, URDF)
Before this commit: robot Carros, 10 links, 9 joints
Joints:
- joint camera_joint: origin xyz=-0.02 0 0.125 rpy=0 0 0 -> xyz=-0.02 0 0.13 rpy=0 0 0

Commit message: Deteccion_carril funcional con interpolacion cuadratica para deteccion de curvas, puntos fijos inferiores en el poligono, reduccion automatica de velocidad.

File: simulacion_ws/src/carro_simulacion/urdf/carro.urdf (robot description, URDF)
Before this commit: robot Carros, 10 links, 9 joints
Joints:
- joint camera_joint: origin xyz=-0.02 0 0.13 rpy=0 0 0 -> xyz=-0.02 0 0.17 rpy=0 0.1 0

Commit message: Manejo correcto en instersecciones, falla en toma de curbatura

File: simulacion_ws/src/carro_simulacion/urdf/carro.urdf (robot description, URDF)
Before this commit: robot Carros, 10 links, 9 joints
Joints:
- joint camera_joint: origin xyz=-0.02 0 0.17 rpy=0 0.1 0 -> xyz=-0.02 0 0.17 rpy=0 0 0

Commit message: actualizacion

File: simulacion_ws/src/carro_simulacion/urdf/carro.urdf (robot description, URDF)
Before this commit: robot Carros, 10 links, 9 joints
Joints:
- joint camera_joint: origin xyz=-0.02 0 0.13 rpy=0 0 0 -> xyz=-0.02 0 0.17 rpy=0 0 0

Commit message: Ultima version del estacionado autonomo

File: simulacion_ws/src/carro_simulacion/urdf/carro.urdf (robot description, URDF)
Before this commit: robot Carros, 10 links, 9 joints
Joints:
- joint lidar_joint: origin xyz=-0.15 0 0.07 rpy=0 0 1.5708 -> xyz=-0.05 0 0.065 rpy=0 0 1.5708
